File: CV-collar.kicad_pcb (KiCad board)
At the start: 2 copper layers, 117 x 54.2 mm, 43 parts, among them J2 MLX90614, J3 UART, J4 BATT_IN, J8 MTHR_I2C, J9 DTR_I2C, Q1 IRLML6401, Q2 AO3401A, SW1 BOOT, SW2 EN, SW3 Addr_SW, SW4 Debug_SW, SW5 PWR, U1 ESP32-WROOM-32, U2 MPU-6050, U3 DS3231M, U4 TPS63900, U5 CW2015CHBD

Commit message: latest before changing to more cost effective design
Parts:
- added U6: MLX90632SLD-DCB-000-RE, footprint:SENSOR-SMD_MLX90632, F.Cu at (268.3, 89.3)
- added U7: LSM6DS3, Package_LGA:LGA-14_3x2.5mm_P0.5mm_LayoutBorder3x4y, F.Cu at (183.8, 83.9)
- BT1: footprint Battery:BatteryHolder_Keystone_103_1x20mm -> Battery:BatteryHolder_Keystone_1060_1x2032
- U3: footprint Package_SO:SOIC-16W_7.5x10.3mm_P1.27mm -> Package_SO:SOIC-8_3.9x4.9mm_P1.27mm
- moved BT1 11.9 mm to (219.5, 100.6)
Connections:
- C4 pad 1: Net-(U2-REGOUT) -> SEN_VCC
- C5 pad 1: Net-(U2-CPOUT) -> unconnected-(C5-Pad1)
- C5 pad 2: GND -> unconnected-(C5-Pad2)
- C6 pad 1: Net-(J2-Pin_4) -> Net-(J9-Pin_3)
- C6 pad 2: Net-(J2-Pin_1) -> Net-(J9-Pin_4)
- J9 pad 1: Net-(J2-Pin_2) -> Net-(J9-Pin_1)
- J9 pad 2: Net-(J2-Pin_3) -> Net-(J9-Pin_2)
- J9 pad 3: Net-(J2-Pin_4) -> Net-(J9-Pin_3)
- J9 pad 4: Net-(J2-Pin_1) -> Net-(J9-Pin_4)
- SW3 pad 1: SEN_VCC -> GND
- SW3 pad 3: GND -> SEN_VCC
Routing:
- net Net-(BT1-+): track 22.0 -> 0.00 mm, vias 1 -> 0
- net GND: track 397.1 -> 419.2 mm, vias 14 -> 15

Commit message: pre jlc
Parts:
- removed C5: 2.2nF, Capacitor_SMD:C_0603_1608Metric
- removed J2: MLX90614, Package_TO_SOT_THT:TO-39-4_Window
- removed SW3: Addr_SW, Button_Switch_SMD:SW_SPDT_PCM12
- removed SW4: Debug_SW, Button_Switch_SMD:SW_SPDT_PCM12
- removed SW5: PWR, Button_Switch_SMD:SW_SPDT_PCM12
- removed U2: MPU-6050, Sensor_Motion:InvenSense_QFN-24_4x4mm_P0.5mm
- added J1: Addr_SW, Connector_PinHeader_2.54mm:PinHeader_1x03_P2.54mm_Vertical, F.Cu at (229.5, 82.2)
- added J5: PWR, Connector_PinHeader_2.54mm:PinHeader_1x02_P2.54mm_Vertical, F.Cu at (229.5, 74.0)
- added J6: Debug_SW, Connector_PinHeader_2.54mm:PinHeader_1x02_P2.54mm_Vertical, F.Cu at (173.9, 99.0)
- J3, J8, J9: footprint Connector_PinHeader_2.54mm:PinHeader_1x04_P2.54mm_Vertical_SMD_Pin1Left -> Connector_PinHeader_2.54mm:PinHeader_1x04_P2.54mm_Vertical
- J4: footprint Connector_PinHeader_2.54mm:PinHeader_1x04_P2.54mm_Vertical_SMD_Pin1Left -> Connector_PinHeader_2.54mm:PinHeader_1x02_P2.54mm_Vertical
- moved J3 76.4 mm to (172.7, 65.4)
- moved R6 47.7 mm to (169.7, 102.0)
- moved U7 23.7 mm to (207.5, 84.8)
- moved C4 23.1 mm to (209.6, 79.2)
- moved U3 22.2 mm to (188.4, 84.1)
- moved Q2 21.4 mm to (219.4, 67.4), turned to 90 degrees
- moved R13 20.8 mm to (196.2, 82.6), turned to 180 degrees
- moved R8 20.0 mm to (188.5, 78.4), turned to -90 degrees
- moved R11 19.5 mm to (197.6, 93.2), turned to 180 degrees
- moved R12 19.5 mm to (201.9, 93.1)
- moved U5 19.5 mm to (199.0, 85.3)
- moved C11 19.5 mm to (197.8, 89.4)
- moved C12 19.5 mm to (201.0, 89.4)
- moved R3 19.0 mm to (188.4, 90.1)
- moved C2 17.7 mm to (185.5, 92.5), turned to -90 degrees
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Connections:
- C6 pad 2: Net-(J9-Pin_4) -> GND
- J9 pad 4: Net-(J9-Pin_4) -> GND
- U3 pad 6: GND -> Net-(BT1-+)
- U3 pad 7: GND -> SDA
- U3 pad 8: GND -> SCL
- U6 pad 3: Net-(J9-Pin_4) -> GND
Routing:
- net GND: track 419.2 -> 29.8 mm, vias 15 -> 13
- net VCC: track 288.8 -> 156.1 mm, vias 3 -> 2
- net GPIO25: track 58.7 -> 174.4 mm, vias 2 -> 0
- net TX: track 105.2 -> 13.7 mm, vias 2 -> 0
- net RX: track 102.6 -> 16.8 mm, vias 2 -> 0
- net GPIO27: track 65.3 -> 8.11 mm, vias 4 -> 0
- net SEN_VCC: track 127.8 -> 74.8 mm, vias 6 -> 2
- net SCL: track 129.7 -> 92.2 mm
- net Net-(BT1-+): track 0.00 -> 33.1 mm, vias 0 -> 2
- net INT/SQW: track 59.5 -> 27.4 mm, vias 2 -> 4
- net SDA: track 118.2 -> 90.5 mm, vias 4 -> 6
- net 3.7V: track 42.0 -> 15.0 mm, vias 0 -> 2
- net Net-(J2-Pin_4): track 23.2 -> 0.00 mm
- net Net-(J9-Pin_1): track 0.00 -> 22.9 mm
- net MPU_INT: track 38.0 -> 54.2 mm, vias 2 -> 4
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- added copper zone on B.Cu, net GND
- added copper zone on F.Cu, net GND
Other:
- board size 117 x 54.2 mm -> 111.8 x 54.2 mm
- board text added: "+"
- board text added: "-"

Commit message: pre jlc
Other:
- board text added: "CV-0.9A"

Commit message: pre jlc
Parts:
- moved C7 9.36 mm to (164.9, 98.5), turned to 0 degrees
- moved C6 2.79 mm to (257.1, 87.1)
Routing:
- net GND: track 29.8 -> 29.9 mm, vias 13 -> 14
Changed lines of the file:
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@@
 	(footprint "Capacitor_SMD:C_0603_1608Metric"
 		(layer "F.Cu")
-		(at 255.04 89.005 -90)
+		(at 257.1 87.125 -90)
 		(descr "Capacitor SMD 0603 (1608 Metric), square (rectangular) end terminal, IPC-7351 nominal, (Body size source: IPC-SM-782 page 76, https://www.pcb-3d.com/wordpress/wp-content/uploads/ipc-sm-782a_amendment_1_and_2.pdf)")
 		(tags "capacitor")
@@
 	(footprint "Capacitor_SMD:C_0603_1608Metric"
 		(layer "F.Cu")
-		(at 173.31 102.68 90)
+		(at 164.93 98.52)
 		(descr "Capacitor SMD 0603 (1608 Metric), square (rectangular) end terminal, IPC-7351 nominal, (Body size source: IPC-SM-782 page 76, https://www.pcb-3d.com/wordpress/wp-content/uploads/ipc-sm-782a_amendment_1_and_2.pdf)")
 		(tags "capacitor")
 		(property "Reference" "C7"
-			(at 0 -1.43 90)
+			(at -0.02 1.59 0)
 			(layer "F.SilkS")
 			(effects
@@
 		)
 		(property "Value" "0.1uF"
-			(at 0 1.43 90)
+			(at 0 1.43 0)
 			(layer "F.Fab")
 			(effects
@@
 		)
 		(property "Datasheet" ""
-			(at 0 0 90)
+			(at 0 0 0)
 			(layer "F.Fab")
 			(hide yes)
@@
 		)
 		(property "Description" "Unpolarized capacitor, small symbol"
-			(at 0 0 90)
+			(at 0 0 0)
 			(layer "F.Fab")
 			(hide yes)
@@
 		)
 		(property "KiLib_Generator" "SMD_2terminal_chip_molded"
-			(at 0 0 90)
+			(at 0 0 0)
 			(layer "F.SilkS")
 			(hide yes)
@@
 		)
 		(property "LCSC Part #" "C1525"
-			(at 0 0 90)
+			(at 0 0 0)
 			(unlocked yes)
 			(layer "F.Fab")
@@
 		)
 		(fp_text user "${REFERENCE}"
-			(at 0 0 90)
+			(at 0 0 0)
 			(layer "F.Fab")
 			(effects
@@
 		)
 		(pad "1" smd roundrect
-			(at -0.775 0 90)
+			(at -0.775 0)
 			(size 0.9 0.95)
 			(layers "F.Cu" "F.Mask" "F.Paste")
@@
 		)
 		(pad "2" smd roundrect
-			(at 0.775 0 90)
+			(at 0.775 0)
 			(size 0.9 0.95)
 			(layers "F.Cu" "F.Mask" "F.Paste")
@@
 	)
 	(segment
+		(start 167.81 99.62)
+		(end 167.9 99.62)
+		(width 0.2)
+		(layer "F.Cu")
+		(net "GND")
+	)
+	(segment
 		(start 251.75 90.69)
 		(end 249.84 90.69)
@@
 	)
 	(via
+		(at 167.81 99.62)
+		(size 0.6)
+		(drill 0.3)
+		(layers "F.Cu" "B.Cu")
+		(free yes)
+		(net "GND")
+	)
+	(via
 		(at 211.59 82.11)
 		(size 0.6)
@@
 		(net "GND")
 	)
+	(segment
+		(start 167.8 99.62)
+		(end 167.81 99.62)
+		(width 0.2)
+		(layer "B.Cu")
+		(net "GND")
+	)
